Commit message: Update screen arm generated assets

File: generated/urdf/face_screen_support_arm.urdf (robot description, URDF)
Before this commit: robot face_screen_support_arm, 8 links, 7 joints
Links:
- link base_link: geometry collision mesh filename=../meshes/base_link.stl scale=0.001 0.001 0.001; visual mesh filename=../visuals/base_disc.stl scale=0.001 0.001 0.001
- link forearm: geometry collision mesh filename=../meshes/forearm.stl scale=0.001 0.001 0.001; visual mesh filename=../visuals/forearm_bar.stl scale=0.001 0.001 0.001
- link screen_pan_link: geometry collision mesh filename=../meshes/screen_pan_link.stl scale=0.001 0.001 0.001; visual mesh filename=../visuals/low_pitch_bridge.stl scale=0.001 0.001 0.001
- link screen_pitch_link: geometry visual mesh filename=../visuals/screen_back_mount.stl scale=0.001 0.001 0.001; visual mesh filename=../visuals/screen_center_marker.stl scale=0.001 0.001 0.001
- link telescopic_slider: geometry collision mesh filename=../meshes/telescopic_slider.stl scale=0.001 0.001 0.001; visual mesh filename=../visuals/inner_tube.stl scale=0.001 0.001 0.001
- link upper_arm: geometry collision mesh filename=../meshes/upper_arm.stl scale=0.001 0.001 0.001; visual mesh filename=../visuals/upper_bar.stl scale=0.001 0.001 0.001
- link yaw_link: geometry collision mesh filename=../meshes/yaw_link.stl scale=0.001 0.001 0.001; visual mesh filename=../visuals/joint2_axis_hint.stl scale=0.001 0.001 0.001
Joints:
- joint joint4_telescopic: limit lower=0 upper=0.45 effort=120 velocity=0.25 -> lower=0 upper=0.28 effort=120 velocity=0.25
- joint joint6_screen_pitch: origin xyz=0.05 0 0.042 rpy=0 0 0 -> xyz=0.07 0 0.042 rpy=0 0 0
- joint screen_center_fixed: origin xyz=0.052 0 0.072 rpy=0 0 0 -> xyz=0.052 0 0.0 rpy=0 0 0
