Commit message: Add face view IK trajectory demo

File: screen_arm/generated/urdf/face_screen_support_arm.urdf (robot description, URDF)
Before this commit: robot face_screen_support_arm, 8 links, 7 joints
Links:
- added link desk_link, mass 25.0; collision mesh filename=../meshes/office_desk.stl scale=0.001 0.001 0.001; visual mesh filename=../meshes/office_desk.stl scale=0.001 0.001 0.001
Joints:
- added joint desk_to_arm_base: type fixed, parent desk_link, child base_link, origin xyz=-0.150 0.000 0.740 rpy=0 0 0
- joint joint2_shoulder_pitch: limit lower=-3.14159 upper=0 effort=35 velocity=1.2 -> lower=-3.49066 upper=0.349066 effort=35 velocity=1.2
- joint joint3_elbow_pitch: limit lower=-2.0944 upper=2.61799 effort=30 velocity=1.2 -> lower=-2.96706 upper=2.96706 effort=30 velocity=1.2
- joint joint5_screen_pan: limit lower=-3.14159 upper=3.14159 effort=8 velocity=2.0 -> lower=-1.74533 upper=1.74533 effort=8 velocity=2.0
